Commit message: added ekf

File: description/ros2_control/diffbot.ros2_control.xacro (robot description, xacro)
@@ -27,4 +27,17 @@
         <state_interface name="velocity"/>
       </joint>
+      <!-- ADD THIS IMU SENSOR BLOCK -->
+      <sensor name="${prefix}imu_sensor">
+        <state_interface name="orientation.x"/>
+        <state_interface name="orientation.y"/>
+        <state_interface name="orientation.z"/>
+        <state_interface name="orientation.w"/>
+        <state_interface name="angular_velocity.x"/>
+        <state_interface name="angular_velocity.y"/>
+        <state_interface name="angular_velocity.z"/>
+        <state_interface name="linear_acceleration.x"/>
+        <state_interface name="linear_acceleration.y"/>
+        <state_interface name="linear_acceleration.z"/>
+      </sensor>
     </ros2_control>
   </xacro:macro>

File: description/urdf/diffbot_description.urdf.xacro (robot description, xacro)
@@ -4,13 +4,13 @@
   <!-- Constants for robot dimensions -->
   <xacro:property name="PI" value="3.1415926535897931"/>
-  <xacro:property name="base_mass" value="0.3" /> <!-- arbitrary value for base mass -->
-  <xacro:property name="base_width" value="0.1" />
-  <xacro:property name="base_length" value="0.1" />
-  <xacro:property name="base_height" value="0.05" />
-  <xacro:property name="wheel_mass" value="0.3" /> <!-- arbitrary value for wheel mass -->
-  <xacro:property name="wheel_len" value="0.020" />
-  <xacro:property name="wheel_radius" value="0.015" />
-  <xacro:property name="caster_wheel_mass" value="0.1" /> <!-- arbitrary value for caster wheel mass -->
-  <xacro:property name="caster_wheel_radius" value="0.015" />
+  <xacro:property name="base_mass" value="1.0" /> <!-- arbitrary value for base mass -->
+  <xacro:property name="base_width" value="0.25" />
+  <xacro:property name="base_length" value="0.25" />
+  <xacro:property name="base_height" value="0.1" />
+  <xacro:property name="wheel_mass" value="0.05" /> <!-- arbitrary value for wheel mass -->
+  <xacro:property name="wheel_len" value="0.026" />
+  <xacro:property name="wheel_radius" value="0.033" />
+  <xacro:property name="caster_wheel_mass" value="0.01" /> <!-- arbitrary value for caster wheel mass -->
+  <xacro:property name="caster_wheel_radius" value="0.016" />
   <xacro:property name="z_offset" value="-${base_height/2}" /> <!-- Space btw top of beam and the each joint -->
   <!-- Base Link -->
